File: hardware/cm4-gpio.kicad_sch (KiCad schematic)
At the start: 6 parts, among them J2 DF40C-100DP-0.4V_51_

Commit message: Cleanup
Other:
- moved on the sheet: J2, R128, R133, R134, R138, R139

Commit message: CleanUP
Connections:
- net SD_DAT4: no longer names the net of J2.68
- net SD_DAT5: no longer names the net of J2.64
- net SD_DAT6 renamed RST_N
- net SD_DAT7: no longer names the net of J2.70
Changed lines of the file:
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@@
-	)
-	(bus_entry
-		(at 97.79 113.03)
-		(size 2.54 2.54)
-		(stroke
-			(width 0)
-			(type default)
-		)
 	)
 	(bus_entry
@@
 	)
 	(bus_entry
-		(at 97.79 115.57)
-		(size 2.54 2.54)
-		(stroke
-			(width 0)
-			(type default)
-		)
-	)
-	(bus_entry
 		(at 97.79 57.15)
 		(size 2.54 2.54)
@@
 	)
 	(bus_entry
-		(at 97.79 105.41)
-		(size 2.54 2.54)
-		(stroke
-			(width 0)
-			(type default)
-		)
-	)
-	(bus_entry
 		(at 97.79 31.75)
 		(size 2.54 2.54)
@@
 	)
 	(bus_entry
-		(at 97.79 110.49)
-		(size 2.54 2.54)
-		(stroke
-			(width 0)
-			(type default)
-		)
-	)
-	(bus_entry
 		(at 46.99 64.77)
 		(size -2.54 2.54)
@@
 		)
 	)
-	(bus
-		(pts
-			(xy 100.33 105.41) (xy 100.33 107.95)
-		)
-		(stroke
-			(width 0)
-			(type default)
-		)
-	)
 	(wire
 		(pts
@@
 		)
 	)
-	(bus
-		(pts
-			(xy 100.33 115.57) (xy 100.33 118.11)
-		)
-		(stroke
-			(width 0)
-			(type default)
-		)
-	)
 	(wire
 		(pts
@@
 		)
 	)
-	(bus
-		(pts
-			(xy 100.33 107.95) (xy 100.33 113.03)
-		)
-		(stroke
-			(width 0)
-			(type default)
-		)
-	)
 	(wire
 		(pts
@@
 		(pts
 			(xy 46.99 64.77) (xy 59.69 64.77)
-		)
-		(stroke
-			(width 0)
-			(type default)
-		)
-	)
-	(bus
-		(pts
-			(xy 100.33 113.03) (xy 100.33 115.57)
 		)
 		(stroke
@@
 		)
 	)
-	(label "SD_DAT4"
-		(at 88.9 110.49 0)
-		(effects
-			(font
-				(size 1.27 1.27)
-			)
-			(justify left bottom)
-		)
-	)
 	(label "GPIO12"
 		(at 46.99 64.77 0)
@@
 		)
 	)
-	(label "SD_DAT7"
-		(at 88.9 113.03 0)
-		(effects
-			(font
-				(size 1.27 1.27)
-			)
-			(justify left bottom)
-		)
-	)
 	(label "ETH3_N"
 		(at 46.99 31.75 0)
@@
 		)
 	)
-	(label "SD_DAT5"
-		(at 88.9 105.41 0)
-		(effects
-			(font
-				(size 1.27 1.27)
-			)
-			(justify left bottom)
-		)
-	)
 	(label "GPIO2"
 		(at 90.17 97.79 0)
@@
 		)
 	)
-	(label "SD_DAT6"
-		(at 88.9 115.57 0)
-		(effects
-			(font
-				(size 1.27 1.27)
-			)
-			(justify left bottom)
-		)
-	)
 	(label "GPIO24"
 		(at 46.99 82.55 0)
@@
 			)
 			(justify left bottom)
+		)
+	)
+	(global_label "RST_N"
+		(shape input)
+		(at 97.79 115.57 0)
+		(fields_autoplaced yes)
+		(effects
+			(font
+				(size 1.27 1.27)
+			)
+			(justify left)
+		)
+		(property "Intersheetrefs" "${INTERSHEET_REFS}"
+			(at 106.5204 115.57 0)
+			(effects
+				(font
+					(size 1.27 1.27)
+				)
+				(justify left)
+				(hide yes)
+			)
+		)
+	)
+	(global_label "PWR_BTN"
+		(shape input)
+		(at 92.71 140.97 0)
+		(fields_autoplaced yes)
+		(effects
+			(font
+				(size 1.27 1.27)
+			)
+			(justify left)
+		)
+		(property "Intersheetrefs" "${INTERSHEET_REFS}"
+			(at 104.2223 140.97 0)
+			(effects
+				(font
+					(size 1.27 1.27)
+				)
+				(justify left)
+				(hide yes)
+			)
 		)
 	)
@@
 		)
 	)
-	(hierarchical_label "PWR_BTN"
-		(shape input)
-		(at 92.71 140.97 0)
-		(effects
-			(font
-				(size 1.27 1.27)
-			)
-			(justify left)
-		)
-	)
