File: hardware/ethernet.kicad_sch (KiCad schematic)
At the start: 92 parts, among them J5 USB_C_Receptacle, Q1 BSS138, Q2 BSS138, U14 KSZ9031RNXCA, U4 GateMate-CCGM1A1, X1 ECS-2520MV-250-xx

Commit message: Improve SerDes routing, tunning ETH pairs, moving parts - fix #31
Parts:
- BTN1, BTN2, BTN3: DigiKey https://www.digikey.com/en/products/detail/panasonic-electr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 -> (none); LCSC (none) -> C231329; MPN (none) -> EVP-AA302K; Mouser Part Number (none) -> 667-EVP-AA302K
- C100, C94: LCSC (none) -> C12530; MPN (none) -> CL05A225MQ5NSNC; Mouser (none) -> https://hr.mouser.com/ProductDetail/Samsung-Electro-Mechani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; Mouser Part Number (none) -> 187-CL05A225MQ5NSNC
- C102, C103, C106, C107, C108, C112, C116, C117, C96, C97: LCSC (none) -> C1525; MPN (none) -> GRM155R60J104KA01D; Mouser (none) -> https://hr.mouser.com/ProductDetail/Murata-Electronics/GRM1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; Mouser Part Number (none) -> 81-GRM155R60J104KA1D
- C104, C105, C109, C114: LCSC (none) -> C15525; MPN (none) -> CL05A106MQ5NUNC; Mouser (none) -> https://hr.mouser.com/ProductDetail/Samsung-Electro-Mechani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; Mouser Part Number (none) -> 187-CL05A106MQ5NUNC
- C110, C111, C113, C119: LCSC (none) -> C15195; MPN (none) -> CL05B103KB5NNNC; Mouser (none) -> https://hr.mouser.com/ProductDetail/Samsung-Electro-Mechani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; Mouser Part Number (none) -> 187-CL05B103KB5NNNC
- C115: LCSC (none) -> C469468; MPN (none) -> CC0402MRX5R6BB475; Mouser (none) -> https://hr.mouser.com/ProductDetail/YAGEO/CC0402MRX5R6BB475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; Mouser Part Number (none) -> 603-CC402MRX5R6BB475
- C118: MPN (none) -> GRM155R60J104KA01D; Mouser (none) -> https://hr.mouser.com/ProductDetail/Murata-Electronics/GRM1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; Mouser Part Number (none) -> 81-GRM155R60J104KA1D; now left out of the parts list
- C95: LCSC (none) -> C16772; MPN (none) -> CL05B224KO5NNNC; Mouser (none) -> https://hr.mouser.com/ProductDetail/Samsung-Electro-Mechani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; Mouser Part Number (none) -> 187-CL05B224KO5NNNC
- C98: LCSC (none) -> C15525; MPN (none) -> CL05A226MQ5N6J8; Mouser (none) -> https://hr.mouser.com/ProductDetail/Samsung-Electro-Mechani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; Mouser Part Number (none) -> 187-CL05A226MQ5N6J8
- D3: Koncar FV002 -> (none); LCSC (none) -> C507914; MNF1_URL www.taiwansemi.com -> (none); MPN BZT52C3V6S -> BZT52C3V6T-7; Mouser 833-BZT52C3V6S-TP -> https://hr.mouser.com/ProductDetail/Diodes-Incorporated/BZT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; Mouser Part Number (none) -> 621-BZT52C3V6T-7; price200_Mouser 0.096$ -> (none)
- D4: LCSC (none) -> C507914; MNF1_URL www.taiwansemi.com -> (none); MPN BZT52C3V6S -> BZT52C3V6T-7; Mouser 833-BZT52C3V6S-TP -> https://hr.mouser.com/ProductDetail/Diodes-Incorporated/BZT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; Mouser Part Number (none) -> 621-BZT52C3V6T-7
- D5, D6, D8: LCSC (none) -> C896167; MPN (none) -> 1N914BWT; Mouser (none) -> https://hr.mouser.com/ProductDetail/onsemi/1N914BWT?qs=2%2F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; Mouser Part Number (none) -> 512-1N914BWT
- D7: LCSC (none) -> C896167; MPN 1N4148WS -> 1N914BWT; Mouser (none) -> https://hr.mouser.com/ProductDetail/onsemi/1N914BWT?qs=2%2F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; Mouser Part Number (none) -> 512-1N914BWT
- FB1, FB2, FB3: LCSC (none) -> C14709; MPN (none) -> BLM18PG121SN1D; Mouser Part Number (none) -> 81-BLM18PG121SN1D
- J5: LCSC (none) -> C37616412; MPN (none) -> USB4215-03-A; Mouser (none) -> https://hr.mouser.com/ProductDetail/GCT/USB4215-03-A?qs=IKk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; Mouser Part Number (none) -> 640-USB4215-03-A; PROD_ID CONN-14122 -> (none)
- Q1, Q2: LCSC (none) -> C40912; MPN (none) -> BSS138; Mouser (none) -> https://hr.mouser.com/ProductDetail/onsemi/BSS138?qs=HK%252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; Mouser Part Number (none) -> 512-BSS138
- R100, R101, R102, R89, R90, R91, R92, R93, R94, R97, R98, R99: LCSC (none) -> C226392; MPN (none) -> AC0402FR-0727RL; Mouser (none) -> https://hr.mouser.com/ProductDetail/YAGEO/RC0402JR-0727RL?q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; Mouser Part Number (none) -> 603-RC0402JR-0727RL
- R103, R47, R55: LCSC (none) -> C144800; MPN (none) -> AC0402FR-0712K1L; Mouser (none) -> https://hr.mouser.com/ProductDetail/YAGEO/AC0402FR-0712K1L?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; Mouser Part Number (none) -> 603-AC0402FR-0712K1L
- R104: MPN (none) -> AC0402FR-0727RL; Mouser (none) -> https://hr.mouser.com/ProductDetail/YAGEO/RC0402JR-0727RL?q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; Mouser Part Number (none) -> 603-RC0402JR-0727RL; now left out of the parts list
- R118: value R300 -> 300R; LCSC (none) -> C100360; MPN (none) -> AC0402FR-07300RL; Mouser (none) -> https://hr.mouser.com/ProductDetail/YAGEO/AC0402FR-07300RL?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; Mouser Part Number (none) -> 603-AC0402FR-07300RL
- R141, R142: LCSC (none) -> C226739; MPN (none) -> AC0402FR-070RL; Mouser (none) -> https://hr.mouser.com/ProductDetail/YAGEO/AC0402FR-070RL?qs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; Mouser Part Number (none) -> 603-AC0402FR-070RL
- R144, R145, R146: value 1K -> 1k; LCSC (none) -> C144789; MPN (none) -> AC0402FR-071KL; Mouser (none) -> https://hr.mouser.com/ProductDetail/YAGEO/AC0402FR-071KL?qs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; Mouser Part Number (none) -> 603-AC0402FR-071KL
- R44, R45: value 27 -> 27R; LCSC (none) -> C226392; MNF1_URL www.yageo.com -> (none); MPN AC0603JR-0727RL -> AC0402FR-0727RL; Mouser (none) -> https://hr.mouser.com/ProductDetail/YAGEO/RC0402JR-0727RL?q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; Mouser Part Number (none) -> 603-RC0402JR-0727RL
- R46, R48: LCSC (none) -> C144789; MPN (none) -> AC0402FR-071KL; Mouser (none) -> https://hr.mouser.com/ProductDetail/YAGEO/AC0402FR-071KL?qs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; Mouser Part Number (none) -> 603-AC0402FR-071KL
- R58: now left out of the parts list
- R61, R62: LCSC (none) -> C25905; MNF1_URL www.yageo.com -> (none); MPN AC0603JR-0727RL -> AC0402FR-7W5K1L; Mouser (none) -> https://hr.mouser.com/ProductDetail/YAGEO/AC0402FR-7W5K1L?q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; Mouser Part Number (none) -> 603-AC0402FR-7W5K1L
- R66, R67, R70, R71, R72, R73, R78, R79, R84, R85, R96: LCSC (none) -> C25900; MPN (none) -> RC0402JR-104K7L; Mouser (none) -> https://hr.mouser.com/ProductDetail/YAGEO/RC0402JR-104K7L?q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; Mouser Part Number (none) -> 603-RC0402JR-104K7L
- R68, R69, R74, R75, R76, R77, R80, R81, R82, R83: now not fitted
- U14: LCSC (none) -> C58758; MPN (none) -> KSZ9031RNXCA; Mouser (none) -> https://hr.mouser.com/ProductDetail/Microchip-Technology/KS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; Mouser Part Number (none) -> 998-KSZ9031RNXCA
- U4: LCSC (none) -> CCGM1A1-BGA324; MPN (none) -> CCGM1A1-BGA324
- X1: MPN (none) -> ECS-2520MV-250-CL-TR; Mouser (none) -> https://hr.mouser.com/ProductDetail/ECS/ECS-2520MV-250-CL-T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; Mouser Part Number (none) -> 520-2520MV-250-CL-TR; now left out of the parts list

Commit message: v0.5 update
Parts:
- added R114: 27R, Resistor_SMD:R_0402_1005Metric, symbol Device:R_Small
- BTN1, BTN2, BTN3: LCSC C231329 -> C79147
- C118, R104, X1: now fitted; now in the parts list
- C98: LCSC C15525 -> C7423886
- Q1, Q2: value BSS138 -> DMG1012T-7; LCSC C40912 -> C2830301; MPN BSS138 -> DMG1012T-7; Mouser https://hr.mouser.com/ProductDetail/onsemi/BSS138?qs=HK%252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 -> https://www.mouser.com/en/ProductDetail/Diodes-Incorporated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; Mouser Part Number 512-BSS138 -> 621-DMG1012T-7
- R100, R101, R102, R44, R45, R89, R90, R91, R92, R93, R94, R97, R98, R99: Mouser https://hr.mouser.com/ProductDetail/YAGEO/RC0402JR-0727RL?q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 -> https://eu.mouser.com/en/ProductDetail/YAGEO/AC0402FR-0727R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; Mouser Part Number 603-RC0402JR-0727RL -> 603-AC0402FR-0727RL
Connections:
- net ETH_CLK: now also R114.2; no longer U4.E16 (IO_EB_A3)
- net at U4.G16 (IO_EA_A8): now also R114.1
