File: hardware/gpio.kicad_sch (KiCad schematic)
At the start: 11 parts, among them U4 GateMate-CCGM1A1

Commit message: Improve SerDes routing, tunning ETH pairs, moving parts - fix #31
Parts:
- C86, C90: LCSC (none) -> C12530; MPN (none) -> CL05A225MQ5NSNC; Mouser (none) -> https://hr.mouser.com/ProductDetail/Samsung-Electro-Mechani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; Mouser Part Number (none) -> 187-CL05A225MQ5NSNC
- C87, C91: LCSC (none) -> C16772; MPN (none) -> CL05B224KO5NNNC; Mouser (none) -> https://hr.mouser.com/ProductDetail/Samsung-Electro-Mechani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; Mouser Part Number (none) -> 187-CL05B224KO5NNNC
- C88, C89, C92, C93: LCSC (none) -> C1525; MPN (none) -> GRM155R60J104KA01D; Mouser (none) -> https://hr.mouser.com/ProductDetail/Murata-Electronics/GRM1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; Mouser Part Number (none) -> 81-GRM155R60J104KA1D
- R115: now not fitted; now left out of the parts list
- R116: LCSC (none) -> C226739; MPN (none) -> AC0402FR-070RL; Mouser (none) -> https://hr.mouser.com/ProductDetail/YAGEO/AC0402FR-070RL?qs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; Mouser Part Number (none) -> 603-AC0402FR-070RL
- U4: LCSC (none) -> CCGM1A1-BGA324; MPN (none) -> CCGM1A1-BGA324
