File: hardware/lvds.kicad_sch (KiCad schematic)
At the start: 52 parts, among them U4 GateMate-CCGM1A1, Y1 ASE2-25.000MHZ-L-C-T

Commit message: Improve SerDes routing, tunning ETH pairs, moving parts - fix #31
Parts:
- C4: LCSC (none) -> C15195; MPN (none) -> CL05B103KB5NNNC; Mouser (none) -> https://hr.mouser.com/ProductDetail/Samsung-Electro-Mechani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; Mouser Part Number (none) -> 187-CL05B103KB5NNNC
- C49, C52, C55, C56: LCSC (none) -> C1525; MPN (none) -> GRM155R60J104KA01D; Mouser (none) -> https://hr.mouser.com/ProductDetail/Murata-Electronics/GRM1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; Mouser Part Number (none) -> 81-GRM155R60J104KA1D
- C50, C53: LCSC (none) -> C15525; MPN (none) -> CL05A226MQ5N6J8; Mouser (none) -> https://hr.mouser.com/ProductDetail/Samsung-Electro-Mechani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; Mouser Part Number (none) -> 187-CL05A226MQ5N6J8
- C51, C54: LCSC (none) -> C12530; MPN (none) -> CL05A225MQ5NSNC; Mouser (none) -> https://hr.mouser.com/ProductDetail/Samsung-Electro-Mechani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; Mouser Part Number (none) -> 187-CL05A225MQ5NSNC
- C59, C60, C61, C62, C63, C64, C65, C66: LCSC (none) -> C16772; MPN (none) -> CL05B224KO5NNNC; Mouser (none) -> https://hr.mouser.com/ProductDetail/Samsung-Electro-Mechani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; Mouser Part Number (none) -> 187-CL05B224KO5NNNC
- D10, D11, D12, D13, D14, D15, D16, D9: LCSC (none) -> C94869; MPN (none) -> LTST-C190KRKT; Mouser (none) -> https://hr.mouser.com/ProductDetail/LITEON/LTST-C190KRKT?qs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; Mouser Part Number (none) -> 859-LTST-C190KRKT
- R121, R122: LCSC (none) -> C137862; MPN (none) -> AF0402FR-074R7L; Mouser (none) -> https://hr.mouser.com/ProductDetail/YAGEO/AF0402FR-074R7L?q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; Mouser Part Number (none) -> 603-AF0402FR-074R7L
- R129, R130, R131, R132, R135, R136, R50, R51, R54: LCSC (none) -> C137918; MPN (none) -> AC0402JR-07150RL; Mouser (none) -> https://hr.mouser.com/ProductDetail/YAGEO/AC0402JR-07150RL?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; Mouser Part Number (none) -> 603-AC0402JR-07150RL
- R59, R63, R64, R65, R86, R87, R88, R95: value R300 -> 300R; LCSC (none) -> C100360; MPN (none) -> AC0402FR-07300RL; Mouser (none) -> https://hr.mouser.com/ProductDetail/YAGEO/AC0402FR-07300RL?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; Mouser Part Number (none) -> 603-AC0402FR-07300RL
- U4: LCSC (none) -> CCGM1A1-BGA324; MPN (none) -> CCGM1A1-BGA324
- Y1: LCSC (none) -> C160454; MNF1_URL https://eu.mouser.com/ProductDetail/ABRACON/ASE2-25.000MHZ-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 -> (none); Mouser (none) -> https://hr.mouser.com/ProductDetail/ABRACON/ASE2-25.000MHZ-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; Mouser Part Number (none) -> 815-ASE2-25.000

Commit message: v0.5 update
Parts:
- C50, C53: LCSC C15525 -> C7423886
- Y1: value ASE2-25.000MHZ-L-C-T -> ECS-3225MV-250-CN-TR; LCSC C160454 -> C5189451; MPN ASE2-25.000MHZ-L-C-T -> ECS-3225MV-250-CN-TR; Mouser https://hr.mouser.com/ProductDetail/ABRACON/ASE2-25.000MHZ-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 -> https://eu.mouser.com/en/ProductDetail/ECS/ECS-3225MV-250-C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; Mouser Part Number 815-ASE2-25.000 -> 520-3225MV-250-CNT
