File: hardware/ulx5m-gs.kicad_sch (KiCad schematic)
At the start: 4 parts

Commit message: Adding fiducials
Parts:
- added FID1, FID2, FID3, FID4: Fiducial, Fiducial:Fiducial_0.5mm_Mask1mm, symbol Mechanical:Fiducial
