File: hardware/panel/ulx5m-gs_panel_checked_v002.kicad_pcb (KiCad board)
At the start: 6 copper layers, 112 x 98 mm, 1262 parts, among them J1 DF40C-100DP-0.4V_51_, J2 DF40C-100DP-0.4V_51_, J3 Vcore_sel, J4 JTAG, J5 USB_C_Receptacle, Q1 BSS138, Q2 BSS138, SW1 CVS-02TB, U1 TLV62569DBV, U10 IS42S16320D-6BLI, U14 KSZ9031RNXCA, U2 TLV62569DBV, U3 MPM3833CGRH-Z, U4 GateMate-CCGM1A1, U5 TLV62569DBV, U6 74LVC1G04GM,115, U7 74LVC2G00HK3-7, U8 74LVC2G00HK3-7, U9 AT25QL321-MBUE-T, X1 ECS-2520MV-250-xx, X2 511FCA100M000BAG, Y1 ASE2-25.000MHZ-L-C-T

Commit message: v0.5 update
Parts:
- removed the BTN1 at (84.5, 123.3)
- removed the BTN1 at (141.5, 123.3)
- removed the BTN1 at (84.5, 81.3)
- removed the BTN1 at (141.5, 81.3)
- removed the BTN2 at (89.7, 82.3)
- removed the BTN2 at (146.7, 124.3)
- removed the BTN2 at (89.7, 124.3)
- removed the BTN2 at (146.7, 82.3)
- removed the BTN3 at (94.6, 81.4)
- removed the BTN3 at (151.6, 123.4)
- removed the BTN3 at (94.6, 123.4)
- removed the BTN3 at (151.6, 81.4)
- removed the C1 at (113.4, 68.2)
- removed the C1 at (113.4, 110.2)
- removed the C1 at (56.4, 110.2)
- removed the C1 at (56.4, 68.2)
- removed the C10 at (106.6, 68.4)
- removed the C10 at (49.6, 68.4)
- removed the C10 at (49.6, 110.4)
- removed the C10 at (106.6, 110.4)
- removed the C100 at (75.1, 74.6)
- removed the C100 at (132.1, 74.6)
- removed the C100 at (132.1, 116.6)
- removed the C100 at (75.1, 116.6)
- removed the C101 at (136.6, 106.0)
- removed the C101 at (136.6, 64.0)
- removed the C101 at (79.6, 64.0)
- removed the C101 at (79.6, 106.0)
- removed the C102 at (136.1, 114.0)
- removed the C102 at (136.1, 72.0)
- removed the C102 at (79.1, 114.0)
- removed the C102 at (79.1, 72.0)
- removed the C103 at (83.0, 116.2)
- removed the C103 at (139.9, 74.2)
- removed the C103 at (139.9, 116.2)
- removed the C103 at (83.0, 74.2)
- removed the C104 at (143.1, 75.3)
- removed the C104 at (143.1, 117.3)
- removed the C104 at (86.1, 117.3)
- removed the C104 at (86.1, 75.3)
- removed the C105 at (149.1, 118.5)
- removed the C105 at (92.1, 76.5)
- removed the C105 at (149.1, 76.5)
- removed the C105 at (92.1, 118.5)
- removed the C106 at (86.0, 73.9)
- removed the C106 at (143.0, 115.9)
- removed the C106 at (86.0, 115.9)
- removed the C106 at (143.0, 73.9)
- removed the C107 at (90.1, 76.5)
- removed the C107 at (90.1, 118.5)
- removed the C107 at (147.1, 76.5)
- removed the C107 at (147.1, 118.5)
- removed the C108 at (86.1, 111.8)
- removed the C108 at (86.1, 69.8)
- removed the C108 at (143.1, 111.8)
- removed the C108 at (143.1, 69.8)
- removed the C109 at (92.6, 69.6)
- removed the C109 at (92.6, 111.6)
- removed the C109 at (149.6, 69.6)
- removed the C109 at (149.6, 111.6)
- removed the C11 at (92.9, 87.1)
- removed the C11 at (149.9, 87.1)
- removed the C11 at (92.9, 129.1)
- removed the C11 at (149.9, 129.1)
- removed the C110 at (91.1, 76.5)
- removed the C110 at (148.1, 118.5)
- removed the C110 at (91.1, 118.5)
- removed the C110 at (148.1, 76.5)
- removed the C111 at (86.0, 114.9)
- removed the C111 at (86.0, 72.9)
- removed the C111 at (143.0, 72.9)
- removed the C111 at (143.0, 114.9)
- removed the C112 at (91.6, 111.6)
- removed the C112 at (148.6, 111.6)
- removed the C112 at (148.6, 69.6)
- removed the C112 at (91.6, 69.6)
- removed the C113 at (143.1, 70.8)
- removed the C113 at (143.1, 112.8)
- removed the C113 at (86.1, 70.8)
- removed the C113 at (86.1, 112.8)
- removed the C114 at (146.6, 69.6)
- removed the C114 at (89.6, 69.6)
- removed the C114 at (146.6, 111.6)
- removed the C114 at (89.6, 111.6)
- removed the C115 at (92.8, 74.2)
- removed the C115 at (149.8, 74.2)
- removed the C115 at (149.8, 116.2)
- removed the C115 at (92.8, 116.2)
- removed the C116 at (90.6, 69.6)
- removed the C116 at (147.6, 111.6)
- removed the C116 at (147.6, 69.6)
- removed the C116 at (90.6, 111.6)
- removed the C117 at (92.8, 73.2)
- removed the C117 at (92.8, 115.2)
- removed the C117 at (149.8, 73.2)
- removed the C117 at (149.8, 115.2)
- removed the C118 at (95.4, 109.9)
- removed the C118 at (152.4, 109.9)
- removed the C118 at (95.4, 67.9)
- removed the C118 at (152.4, 67.9)
- removed the C119 at (149.8, 72.2)
- removed the C119 at (92.8, 114.2)
- removed the C119 at (149.8, 114.2)
- removed the C119 at (92.8, 72.2)
- removed the C120 at (117.9, 69.5)
- removed the C120 at (60.9, 69.5)
- removed the C120 at (60.9, 111.5)
- removed the C120 at (117.9, 111.5)
- removed the C121 at (113.9, 120.9)
- removed the C121 at (56.9, 120.9)
- removed the C121 at (113.9, 78.9)
- removed the C121 at (56.9, 78.9)
- removed the C122 at (139.9, 72.3)
- removed the C122 at (139.9, 114.3)
- removed the C122 at (82.9, 114.3)
- removed the C122 at (82.9, 72.3)
- removed the C123 at (137.3, 124.7)
- removed the C123 at (80.3, 124.7)
- removed the C123 at (80.3, 82.7)
- removed the C123 at (137.3, 82.7)
- removed the C124 at (78.3, 106.1)
- removed the C124 at (135.3, 106.1)
- removed the C124 at (78.3, 64.1)
- removed the C124 at (135.3, 64.1)
- removed the C125 at (140.9, 72.3)
- removed the C125 at (140.9, 114.3)
- removed the C125 at (83.9, 72.3)
- removed the C125 at (83.9, 114.3)
- removed the C126 at (134.2, 133.9)
- removed the C126 at (77.2, 133.9)
- removed the C126 at (134.2, 91.9)
- removed the C126 at (77.2, 91.9)
- removed the C127 at (135.0, 85.4)
- removed the C127 at (78.0, 127.4)
- removed the C127 at (78.0, 85.4)
- removed the C127 at (135.0, 127.4)
- removed the C128 at (84.1, 81.8)
- removed the C128 at (84.1, 123.8)
- removed the C128 at (141.1, 123.8)
- removed the C128 at (141.1, 81.8)
- removed the C129 at (126.8, 133.5)
- removed the C129 at (126.8, 91.5)
- removed the C129 at (69.8, 91.5)
- removed the C129 at (69.8, 133.5)
- removed the C13 at (137.8, 74.1)
- removed the C13 at (80.8, 74.1)
- removed the C13 at (80.8, 116.1)
- removed the C13 at (137.8, 116.1)
- removed the C130 at (70.8, 133.5)
- removed the C130 at (127.8, 91.5)
- removed the C130 at (70.8, 91.5)
- removed the C130 at (127.8, 133.5)
- removed the C131 at (75.8, 95.0)
- removed the C131 at (132.8, 137.0)
- removed the C131 at (132.8, 95.0)
- removed the C131 at (75.8, 137.0)
- removed the C132 at (76.7, 96.2)
- removed the C132 at (133.7, 96.2)
- removed the C132 at (76.7, 138.2)
- removed the C132 at (133.7, 138.2)
- removed the C133 at (79.1, 88.5)
- removed the C133 at (136.1, 130.5)
- removed the C133 at (136.1, 88.5)
- removed the C133 at (79.1, 130.5)
- removed the C134 at (68.8, 91.5)
- removed the C134 at (125.8, 91.5)
- removed the C134 at (125.8, 133.5)
- removed the C134 at (68.8, 133.5)
- removed the C135 at (124.9, 91.5)
- removed the C135 at (67.9, 133.5)
- removed the C135 at (67.9, 91.5)
- removed the C135 at (124.9, 133.5)
- removed the C136 at (73.7, 96.2)
- removed the C136 at (130.7, 138.2)
- removed the C136 at (73.7, 138.2)
- removed the C136 at (130.7, 96.2)
- removed the C137 at (131.6, 96.2)
- removed the C137 at (74.6, 96.2)
- removed the C137 at (74.6, 138.2)
- removed the C137 at (131.6, 138.2)
- removed the C138 at (79.6, 80.3)
- removed the C138 at (79.6, 122.3)
- removed the C138 at (136.6, 122.3)
- removed the C138 at (136.6, 80.3)
- removed the C14 at (57.0, 119.0)
- removed the C14 at (57.0, 77.0)
- removed the C14 at (114.0, 77.0)
- removed the C14 at (114.0, 119.0)
- removed the C140 at (103.4, 128.7)
- removed the C140 at (46.4, 86.7)
- removed the C140 at (103.4, 86.7)
- removed the C140 at (46.4, 128.7)
- removed the C141 at (45.8, 127.3)
- removed the C141 at (102.8, 85.3)
- removed the C141 at (102.8, 127.3)
- removed the C141 at (45.8, 85.3)
- removed the C15 at (69.6, 122.9)
- removed the C15 at (126.6, 80.9)
- removed the C15 at (126.6, 122.9)
- removed the C15 at (69.6, 80.9)
- removed the C16 at (59.8, 111.5)
- removed the C16 at (116.8, 111.5)
- removed the C16 at (59.8, 69.5)
- removed the C16 at (116.8, 69.5)
- removed the C17 at (132.2, 121.0)
- removed the C17 at (75.2, 121.0)
- removed the C17 at (132.2, 79.0)
- removed the C17 at (75.2, 79.0)
- removed the C18 at (75.2, 119.2)
- removed the C18 at (132.2, 119.2)
- removed the C18 at (132.2, 77.2)
- removed the C18 at (75.2, 77.2)
- removed the C2 at (142.2, 60.2)
- removed the C2 at (85.2, 102.2)
- removed the C2 at (142.2, 102.2)
- removed the C2 at (85.2, 60.2)
- removed the C21 at (128.9, 77.2)
- removed the C21 at (72.0, 77.2)
- removed the C21 at (128.9, 119.2)
- removed the C21 at (72.0, 119.2)
- removed the C22 at (129.0, 78.1)
- removed the C22 at (129.0, 120.1)
- removed the C22 at (72.0, 78.1)
- removed the C22 at (72.0, 120.1)
- removed the C23 at (72.0, 80.9)
- removed the C23 at (129.0, 122.9)
- removed the C23 at (72.0, 122.9)
- removed the C23 at (129.0, 80.9)
- removed the C24 at (93.4, 125.6)
- removed the C24 at (150.4, 83.6)
- removed the C24 at (93.4, 83.6)
- removed the C24 at (150.4, 125.6)
- removed the C26 at (126.6, 120.1)
- removed the C26 at (69.6, 120.1)
- removed the C26 at (126.6, 78.1)
- removed the C26 at (69.6, 78.1)
- removed the C27 at (129.0, 79.1)
- removed the C27 at (129.0, 121.1)
- removed the C27 at (72.0, 79.1)
- removed the C27 at (72.0, 121.1)
- removed the C28 at (75.2, 120.1)
- removed the C28 at (132.2, 78.1)
- removed the C28 at (75.2, 78.1)
- removed the C28 at (132.2, 120.1)
- removed the C29 at (92.3, 125.6)
- removed the C29 at (92.3, 83.6)
- removed the C29 at (149.3, 83.6)
- removed the C29 at (149.3, 125.6)
- removed the C3 at (48.6, 70.8)
- removed the C3 at (105.7, 112.8)
- removed the C3 at (48.6, 112.8)
- removed the C3 at (105.7, 70.8)
- removed the C31 at (75.2, 122.0)
- removed the C31 at (132.2, 122.0)
- removed the C31 at (75.2, 80.0)
- removed the C31 at (132.2, 80.0)
- removed the C32 at (126.6, 79.0)
- removed the C32 at (69.6, 79.0)
- removed the C32 at (69.6, 121.0)
- removed the C32 at (126.6, 121.0)
- removed the C33 at (130.0, 111.2)
- removed the C33 at (73.0, 69.2)
- removed the C33 at (130.0, 69.2)
- removed the C33 at (73.0, 111.2)
- removed the C34 at (71.9, 109.2)
- removed the C34 at (71.9, 67.2)
- removed the C34 at (128.9, 67.2)
- removed the C34 at (128.9, 109.2)
- removed the C35 at (69.6, 121.9)
- removed the C35 at (69.6, 79.9)
- removed the C35 at (126.6, 79.9)
- removed the C35 at (126.6, 121.9)
- removed the C36 at (77.3, 64.1)
- removed the C36 at (77.3, 106.1)
- removed the C36 at (134.3, 106.1)
- removed the C36 at (134.3, 64.1)
- removed the C37 at (57.5, 109.3)
- removed the C37 at (114.5, 109.3)
- removed the C37 at (114.5, 67.3)
- removed the C37 at (57.5, 67.3)
- removed the C38 at (132.2, 81.0)
- removed the C38 at (75.2, 81.0)
- removed the C38 at (132.2, 123.0)
- removed the C38 at (75.2, 123.0)
- removed the C39 at (114.0, 78.0)
- removed the C39 at (114.0, 120.0)
- removed the C39 at (57.0, 78.0)
- removed the C39 at (57.0, 120.0)
- removed the C4 at (143.0, 122.6)
- removed the C4 at (143.0, 80.6)
- removed the C4 at (86.0, 122.6)
- removed the C4 at (86.0, 80.6)
- removed the C40 at (126.6, 119.2)
- removed the C40 at (69.6, 119.2)
- removed the C40 at (126.6, 77.2)
- removed the C40 at (69.6, 77.2)
- removed the C41 at (129.0, 122.0)
- removed the C41 at (72.0, 122.0)
- removed the C41 at (72.0, 80.0)
- removed the C41 at (129.0, 80.0)
- removed the C42 at (140.2, 129.7)
- removed the C42 at (83.2, 87.7)
- removed the C42 at (83.2, 129.7)
- removed the C42 at (140.2, 87.7)
- removed the C43 at (63.7, 85.1)
- removed the C43 at (63.7, 127.1)
- removed the C43 at (120.7, 85.1)
- removed the C43 at (120.7, 127.1)
- removed the C44 at (122.7, 85.1)
- removed the C44 at (122.7, 127.1)
- removed the C44 at (65.7, 127.1)
- removed the C44 at (65.7, 85.1)
- removed the C45 at (64.7, 127.1)
- removed the C45 at (121.7, 85.1)
- removed the C45 at (64.7, 85.1)
- removed the C45 at (121.7, 127.1)
- removed the C47 at (136.6, 62.1)
- removed the C47 at (79.6, 104.2)
- removed the C47 at (136.6, 104.2)
- removed the C47 at (79.6, 62.1)
- removed the C48 at (113.8, 125.7)
- removed the C48 at (113.8, 83.7)
- removed the C48 at (56.8, 83.7)
- removed the C48 at (56.8, 125.7)
- removed the C49 at (123.9, 84.8)
- removed the C49 at (66.9, 126.8)
- removed the C49 at (123.9, 126.8)
- removed the C49 at (66.9, 84.8)
- removed the C50 at (70.5, 82.2)
- removed the C50 at (127.5, 82.2)
- removed the C50 at (70.5, 124.2)
- removed the C50 at (127.5, 124.2)
- removed the C51 at (71.5, 82.3)
- removed the C51 at (128.5, 82.3)
- removed the C51 at (71.5, 124.3)
- removed the C51 at (128.5, 124.3)
- removed the C52 at (72.4, 124.3)
- removed the C52 at (129.4, 82.3)
- removed the C52 at (72.4, 82.3)
- removed the C52 at (129.4, 124.3)
- removed the C53 at (75.2, 82.0)
- removed the C53 at (132.2, 82.0)
- removed the C53 at (75.2, 124.0)
- removed the C53 at (132.2, 124.0)
- removed the C54 at (74.5, 85.5)
- removed the C54 at (131.5, 85.5)
- removed the C54 at (74.5, 127.5)
- removed the C54 at (131.5, 127.5)
- removed the C55 at (132.5, 127.5)
- removed the C55 at (75.5, 127.5)
- removed the C55 at (75.5, 85.5)
- removed the C55 at (132.5, 85.5)
- removed the C56 at (136.4, 127.1)
- removed the C56 at (79.4, 85.1)
- removed the C56 at (136.4, 85.1)
- removed the C56 at (79.4, 127.1)
- removed the C57 at (114.6, 123.0)
- removed the C57 at (57.6, 123.0)
- removed the C57 at (57.6, 81.0)
- removed the C57 at (114.6, 81.0)
- removed the C58 at (68.2, 123.5)
- removed the C58 at (125.2, 123.5)
- removed the C58 at (125.2, 81.5)
- removed the C58 at (68.2, 81.5)
- removed the C59 at (61.0, 137.7)
- removed the C59 at (118.0, 95.7)
- removed the C59 at (118.0, 137.7)
- removed the C59 at (61.0, 95.7)
- removed the C6 at (141.7, 105.6)
- removed the C6 at (84.7, 63.6)
- removed the C6 at (84.7, 105.6)
- removed the C6 at (141.7, 63.6)
- removed the C60 at (117.0, 137.7)
- removed the C60 at (60.0, 137.7)
- removed the C60 at (117.0, 95.7)
- removed the C60 at (60.0, 95.7)
- removed the C61 at (120.0, 137.7)
- removed the C61 at (120.0, 95.7)
- removed the C61 at (63.0, 95.7)
- removed the C61 at (63.0, 137.7)
- removed the C62 at (62.0, 137.7)
- removed the C62 at (62.0, 95.7)
- removed the C62 at (119.0, 95.7)
- removed the C62 at (119.0, 137.7)
- removed the C63 at (64.9, 137.7)
- removed the C63 at (121.9, 95.7)
- removed the C63 at (121.9, 137.7)
- removed the C63 at (64.9, 95.7)
- removed the C64 at (63.9, 137.7)
- removed the C64 at (120.9, 137.7)
- removed the C64 at (120.9, 95.7)
- removed the C64 at (63.9, 95.7)
- removed the C65 at (116.1, 137.7)
- removed the C65 at (59.1, 137.7)
- removed the C65 at (59.1, 95.7)
- removed the C65 at (116.1, 95.7)
- removed the C66 at (58.1, 95.7)
- removed the C66 at (58.1, 137.7)
- removed the C66 at (115.1, 95.7)
- removed the C66 at (115.1, 137.7)
- removed the C7 at (106.2, 109.3)
- removed the C7 at (49.2, 109.3)
- removed the C7 at (49.2, 67.3)
- removed the C7 at (106.2, 67.3)
- removed the C75 at (59.5, 81.0)
- removed the C75 at (116.5, 123.0)
- removed the C75 at (116.5, 81.0)
- removed the C75 at (59.5, 123.0)
- removed the C76 at (60.5, 81.0)
- removed the C76 at (117.5, 81.0)
- removed the C76 at (60.5, 123.0)
- removed the C76 at (117.5, 123.0)
- removed the C77 at (68.7, 117.9)
- removed the C77 at (125.7, 117.9)
- removed the C77 at (68.7, 75.9)
- removed the C77 at (125.7, 75.9)
- removed the C78 at (65.3, 117.8)
- removed the C78 at (122.3, 117.8)
- removed the C78 at (65.3, 75.8)
- removed the C78 at (122.3, 75.8)
- removed the C79 at (122.6, 72.6)
- removed the C79 at (122.6, 114.6)
- removed the C79 at (65.6, 114.6)
- removed the C79 at (65.6, 72.6)
- removed the C8 at (85.7, 63.6)
- removed the C8 at (85.7, 105.6)
- removed the C8 at (142.7, 63.6)
- removed the C8 at (142.7, 105.6)
- removed the C80 at (108.7, 78.5)
- removed the C80 at (51.7, 120.5)
- removed the C80 at (51.7, 78.5)
- removed the C80 at (108.7, 120.5)
- removed the C85 at (137.8, 105.5)
- removed the C85 at (80.8, 63.5)
- removed the C85 at (80.8, 105.5)
- removed the C85 at (137.8, 63.5)
- removed the C86 at (50.9, 82.4)
- removed the C86 at (50.9, 124.4)
- removed the C86 at (107.9, 124.4)
- removed the C86 at (107.9, 82.4)
- removed the C87 at (55.5, 119.5)
- removed the C87 at (112.5, 119.5)
- removed the C87 at (112.5, 77.5)
- removed the C87 at (55.5, 77.5)
- removed the C88 at (48.1, 84.5)
- removed the C88 at (105.1, 84.5)
- removed the C88 at (48.1, 126.5)
- removed the C88 at (105.1, 126.5)
- removed the C89 at (105.1, 124.6)
- removed the C89 at (48.1, 82.6)
- removed the C89 at (105.1, 82.6)
- removed the C89 at (48.1, 124.6)
- removed the C9 at (48.2, 67.3)
- removed the C9 at (105.2, 67.3)
- removed the C9 at (48.2, 109.3)
- removed the C9 at (105.2, 109.3)
- removed the C90 at (46.6, 82.6)
- removed the C90 at (103.7, 82.6)
- removed the C90 at (46.6, 124.6)
- removed the C90 at (103.7, 124.6)
- removed the C91 at (111.3, 119.5)
- removed the C91 at (54.3, 119.5)
- removed the C91 at (111.3, 77.5)
- removed the C91 at (54.3, 77.5)
- removed the C92 at (113.5, 123.0)
- removed the C92 at (113.5, 81.0)
- removed the C92 at (56.5, 81.0)
- removed the C92 at (56.5, 123.0)
- removed the C93 at (53.9, 125.7)
- removed the C93 at (110.8, 125.7)
- removed the C93 at (110.8, 83.7)
- removed the C93 at (53.9, 83.7)
- removed the C94 at (50.5, 87.2)
- removed the C94 at (107.5, 129.2)
- removed the C94 at (107.5, 87.2)
- removed the C94 at (50.5, 129.2)
- removed the C95 at (81.5, 78.4)
- removed the C95 at (81.5, 120.4)
- removed the C95 at (138.5, 78.4)
- removed the C95 at (138.5, 120.4)
- removed the C96 at (80.5, 120.4)
- removed the C96 at (137.5, 120.4)
- removed the C96 at (137.5, 78.4)
- removed the C96 at (80.5, 78.4)
- removed the C97 at (79.5, 78.4)
- removed the C97 at (79.5, 120.4)
- removed the C97 at (136.5, 78.4)
- removed the C97 at (136.5, 120.4)
- removed the C98 at (133.0, 117.5)
- removed the C98 at (133.0, 75.5)
- removed the C98 at (76.0, 117.5)
- removed the C98 at (76.0, 75.5)
- removed the C99 at (61.1, 107.0)
- removed the C99 at (118.1, 107.0)
- removed the C99 at (118.1, 65.0)
- removed the C99 at (61.1, 65.0)
- removed the D1 at (109.0, 95.1)
- removed the D1 at (52.0, 95.1)
- removed the D1 at (52.0, 137.1)
- removed the D1 at (109.0, 137.1)
- removed the D10 at (85.7, 129.7)
- removed the D10 at (142.7, 87.7)
- removed the D10 at (142.7, 129.7)
- removed the D10 at (85.7, 87.7)
- removed the D11 at (144.3, 87.7)
- removed the D11 at (87.3, 87.7)
- removed the D11 at (87.3, 129.7)
- removed the D11 at (144.3, 129.7)
- removed the D12 at (88.9, 129.7)
- removed the D12 at (145.9, 87.7)
- removed the D12 at (145.9, 129.7)
- removed the D12 at (88.9, 87.7)
- removed the D13 at (90.5, 129.7)
- removed the D13 at (147.5, 87.7)
- removed the D13 at (147.5, 129.7)
- removed the D13 at (90.5, 87.7)
- removed the D14 at (149.1, 129.7)
- removed the D14 at (149.1, 87.7)
- removed the D14 at (92.1, 129.7)
- removed the D14 at (92.1, 87.7)
- removed the D15 at (93.7, 129.7)
- removed the D15 at (150.7, 129.7)
- removed the D15 at (150.7, 87.7)
- removed the D15 at (93.7, 87.7)
- removed the D16 at (95.3, 129.7)
- removed the D16 at (152.3, 129.7)
- removed the D16 at (95.3, 87.7)
- removed the D16 at (152.3, 87.7)
- removed the D2 at (56.1, 137.1)
- removed the D2 at (113.1, 137.1)
- removed the D2 at (113.1, 95.1)
- removed the D2 at (56.1, 95.1)
- removed the D3 at (143.9, 129.2)
- removed the D3 at (143.9, 87.2)
- removed the D3 at (86.9, 129.2)
- removed the D3 at (86.9, 87.2)
- removed the D4 at (85.5, 87.2)
- removed the D4 at (142.5, 87.2)
- removed the D4 at (142.5, 129.2)
- removed the D4 at (85.5, 129.2)
- removed the D5 at (125.7, 138.6)
- removed the D5 at (125.7, 96.6)
- removed the D5 at (68.7, 96.6)
- removed the D5 at (68.7, 138.6)
- removed the D6 at (71.2, 138.7)
- removed the D6 at (71.2, 96.7)
- removed the D6 at (128.2, 138.7)
- removed the D6 at (128.2, 96.7)
- removed the D7 at (131.4, 131.2)
- removed the D7 at (74.4, 131.2)
- removed the D7 at (131.4, 89.2)
- removed the D7 at (74.4, 89.2)
- removed the D8 at (77.9, 130.9)
- removed the D8 at (77.9, 88.9)
- removed the D8 at (134.9, 88.9)
- removed the D8 at (134.9, 130.9)
- removed the D9 at (84.1, 87.7)
- removed the D9 at (84.1, 129.7)
- removed the D9 at (141.1, 129.7)
- removed the D9 at (141.1, 87.7)
- removed the FB1 at (92.7, 67.0)
- removed the FB1 at (149.7, 67.0)
- removed the FB1 at (92.7, 109.0)
- removed the FB1 at (149.7, 109.0)
- removed the FB2 at (147.3, 67.6)
- removed the FB2 at (90.3, 109.6)
- removed the FB2 at (90.3, 67.6)
- removed the FB2 at (147.3, 109.6)
- removed the FB3 at (94.7, 115.6)
- removed the FB3 at (151.7, 115.6)
- removed the FB3 at (151.7, 73.6)
- removed the FB3 at (94.7, 73.6)
- removed the G*** at (51.2, 115.3)
- removed the G*** at (122.0, 90.7)
- removed the G*** at (65.0, 90.7)
- removed the G*** at (109.4, 127.3)
- removed the G*** at (52.4, 85.3)
- removed the G*** at (65.0, 132.7)
- removed the G*** at (108.2, 115.3)
- removed the G*** at (122.0, 132.7)
- removed the G*** at (52.4, 127.3)
- removed the G*** at (51.2, 73.3)
- removed the G*** at (109.4, 85.3)
- removed the G*** at (108.2, 73.3)
- removed the H1 at (103.0, 103.5)
- removed the H1 at (103.0, 61.5)
- removed the H1 at (46.0, 61.5)
- removed the H1 at (46.0, 103.5)
- removed the H2 at (151.0, 103.5)
- removed the H2 at (151.0, 61.5)
- removed the H2 at (94.0, 61.5)
- removed the H2 at (94.0, 103.5)
- removed the H3 at (103.0, 136.5)
- removed the H3 at (46.0, 94.5)
- removed the H3 at (46.0, 136.5)
- removed the H3 at (103.0, 94.5)
- removed the H4 at (94.0, 94.5)
- removed the H4 at (151.0, 136.5)
- removed the H4 at (151.0, 94.5)
- removed the H4 at (94.0, 136.5)
- removed the J1 at (67.5, 95.0)
- removed the J1 at (124.5, 95.0)
- removed the J1 at (124.5, 137.0)
- removed the J1 at (67.5, 137.0)
- removed the J2 at (67.5, 61.0)
- removed the J2 at (124.5, 103.0)
- removed the J2 at (124.5, 61.0)
- removed the J2 at (67.5, 103.0)
- removed the J3 at (54.8, 102.9)
- removed the J3 at (111.8, 60.9)
- removed the J3 at (111.8, 102.9)
- removed the J3 at (54.8, 60.9)
- removed the J4 at (57.8, 132.3)
- removed the J4 at (114.8, 132.3)
- removed the J4 at (114.8, 90.3)
- removed the J4 at (57.8, 90.3)
- removed the J5 at (141.6, 90.7)
- removed the J5 at (84.6, 90.7)
- removed the J5 at (141.6, 132.7)
- removed the J5 at (84.6, 132.7)
- removed the JP1 at (117.5, 85.0)
- removed the JP1 at (60.5, 85.0)
- removed the JP1 at (60.5, 127.0)
- removed the JP1 at (117.5, 127.0)
- removed the L1 at (145.2, 106.0)
- removed the L1 at (88.2, 106.0)
- removed the L1 at (145.2, 64.0)
- removed the L1 at (88.2, 64.0)
- removed the L2 at (45.7, 108.8)
- removed the L2 at (102.7, 108.8)
- removed the L2 at (45.7, 66.8)
- removed the L2 at (102.7, 66.8)
- removed the L3 at (89.9, 125.2)
- removed the L3 at (146.9, 83.2)
- removed the L3 at (89.9, 83.2)
- removed the L3 at (146.9, 125.2)
- removed the LoGo_opencologne at (143.6, 62.8)
- removed the LoGo_opencologne at (143.6, 104.8)
- removed the LoGo_opencologne at (86.6, 104.8)
- removed the LoGo_opencologne at (86.6, 62.8)
- removed the Q1 at (87.0, 109.4)
- removed the Q1 at (144.1, 67.4)
- removed the Q1 at (144.1, 109.4)
- removed the Q1 at (87.0, 67.4)
- removed the Q2 at (83.3, 67.4)
- removed the Q2 at (140.3, 109.4)
- removed the Q2 at (140.3, 67.4)
- removed the Q2 at (83.3, 109.4)
- removed the R1 at (55.6, 70.4)
- removed the R1 at (112.6, 112.4)
- removed the R1 at (112.6, 70.4)
- removed the R1 at (55.6, 112.4)
- removed the R10 at (82.5, 105.9)
- removed the R10 at (139.5, 63.9)
- removed the R10 at (82.5, 63.9)
- removed the R10 at (139.5, 105.9)
- removed the R100 at (145.0, 78.7)
- removed the R100 at (145.0, 120.7)
- removed the R100 at (88.0, 78.7)
- removed the R100 at (88.0, 120.7)
- removed the R101 at (144.0, 120.7)
- removed the R101 at (87.0, 78.7)
- removed the R101 at (87.0, 120.7)
- removed the R101 at (144.0, 78.7)
- removed the R102 at (92.3, 120.7)
- removed the R102 at (149.3, 120.7)
- removed the R102 at (92.3, 78.7)
- removed the R102 at (149.3, 78.7)
- removed the R103 at (151.1, 68.9)
- removed the R103 at (94.1, 68.9)
- removed the R103 at (94.1, 110.9)
- removed the R103 at (151.1, 110.9)
- removed the R104 at (151.1, 112.8)
- removed the R104 at (94.1, 112.8)
- removed the R104 at (94.1, 70.8)
- removed the R104 at (151.1, 70.8)
- removed the R105 at (138.2, 128.5)
- removed the R105 at (81.2, 86.5)
- removed the R105 at (138.2, 86.5)
- removed the R105 at (81.2, 128.5)
- removed the R106 at (141.1, 125.0)
- removed the R106 at (84.1, 83.0)
- removed the R106 at (84.1, 125.0)
- removed the R106 at (141.1, 83.0)
- removed the R107 at (68.3, 136.9)
- removed the R107 at (125.3, 136.9)
- removed the R107 at (68.3, 94.9)
- removed the R107 at (125.3, 94.9)
- removed the R108 at (127.7, 90.5)
- removed the R108 at (70.7, 132.6)
- removed the R108 at (127.7, 132.6)
- removed the R108 at (70.7, 90.5)
- removed the R109 at (131.4, 133.5)
- removed the R109 at (74.4, 91.5)
- removed the R109 at (74.4, 133.5)
- removed the R109 at (131.4, 91.5)
- removed the R11 at (108.2, 67.7)
- removed the R11 at (108.2, 109.7)
- removed the R11 at (51.2, 67.7)
- removed the R11 at (51.2, 109.7)
- removed the R110 at (68.9, 132.1)
- removed the R110 at (125.9, 90.1)
- removed the R110 at (125.9, 132.1)
- removed the R110 at (68.9, 90.1)
- removed the R111 at (77.8, 125.6)
- removed the R111 at (77.8, 83.6)
- removed the R111 at (134.8, 83.6)
- removed the R111 at (134.8, 125.6)
- removed the R112 at (80.8, 131.3)
- removed the R112 at (137.8, 131.3)
- removed the R112 at (137.8, 89.3)
- removed the R112 at (80.8, 89.3)
- removed the R113 at (81.1, 130.3)
- removed the R113 at (138.1, 130.3)
- removed the R113 at (138.1, 88.3)
- removed the R113 at (81.1, 88.3)
- removed the R115 at (102.2, 126.1)
- removed the R115 at (45.2, 84.1)
- removed the R115 at (45.2, 126.1)
- removed the R115 at (102.2, 84.1)
- removed the R116 at (102.2, 83.1)
- removed the R116 at (45.2, 125.1)
- removed the R116 at (45.2, 83.1)
- removed the R116 at (102.2, 125.1)
- removed the R118 at (93.6, 78.7)
- removed the R118 at (150.6, 120.7)
- removed the R118 at (93.6, 120.7)
- removed the R118 at (150.6, 78.7)
- removed the R12 at (54.8, 107.4)
- removed the R12 at (54.8, 65.4)
- removed the R12 at (111.8, 107.4)
- removed the R12 at (111.8, 65.4)
- removed the R121 at (65.1, 86.5)
- removed the R121 at (122.1, 128.5)
- removed the R121 at (122.1, 86.5)
- removed the R121 at (65.1, 128.5)
- removed the R122 at (82.0, 127.3)
- removed the R122 at (139.0, 85.3)
- removed the R122 at (82.0, 85.3)
- removed the R122 at (139.0, 127.3)
- removed the R123 at (62.7, 127.1)
- removed the R123 at (62.7, 85.1)
- removed the R123 at (119.7, 127.1)
- removed the R123 at (119.7, 85.1)
- removed the R128 at (120.4, 67.0)
- removed the R128 at (63.4, 109.0)
- removed the R128 at (63.4, 67.0)
- removed the R128 at (120.4, 109.0)
- removed the R129 at (69.4, 83.7)
- removed the R129 at (126.4, 83.7)
- removed the R129 at (69.4, 125.7)
- removed the R129 at (126.4, 125.7)
- removed the R13 at (109.8, 107.3)
- removed the R13 at (52.8, 65.3)
- removed the R13 at (109.8, 65.3)
- removed the R13 at (52.8, 107.3)
- removed the R130 at (126.7, 133.7)
- removed the R130 at (126.7, 91.7)
- removed the R130 at (69.7, 133.7)
- removed the R130 at (69.7, 91.7)
- removed the R131 at (68.2, 134.4)
- removed the R131 at (125.2, 134.4)
- removed the R131 at (68.2, 92.4)
- removed the R131 at (125.2, 92.4)
- removed the R132 at (69.6, 87.2)
- removed the R132 at (126.6, 87.2)
- removed the R132 at (126.6, 129.2)
- removed the R132 at (69.6, 129.2)
- removed the R134 at (119.4, 67.0)
- removed the R134 at (119.4, 109.0)
- removed the R134 at (62.4, 109.0)
- removed the R134 at (62.4, 67.0)
- removed the R135 at (127.9, 84.2)
- removed the R135 at (127.9, 126.2)
- removed the R135 at (70.9, 126.2)
- removed the R135 at (70.9, 84.2)
- removed the R136 at (115.8, 135.6)
- removed the R136 at (115.8, 93.6)
- removed the R136 at (58.8, 93.6)
- removed the R136 at (58.8, 135.6)
- removed the R138 at (118.4, 109.0)
- removed the R138 at (118.4, 67.0)
- removed the R138 at (61.4, 109.0)
- removed the R138 at (61.4, 67.0)
- removed the R139 at (116.4, 67.0)
- removed the R139 at (116.4, 109.0)
- removed the R139 at (59.4, 67.0)
- removed the R139 at (59.4, 109.0)
- removed the R14 at (113.3, 64.8)
- removed the R14 at (56.3, 64.8)
- removed the R14 at (56.3, 106.8)
- removed the R14 at (113.3, 106.8)
- removed the R141 at (136.5, 93.3)
- removed the R141 at (79.5, 135.3)
- removed the R141 at (79.5, 93.3)
- removed the R141 at (136.5, 135.3)
- removed the R142 at (78.2, 91.1)
- removed the R142 at (135.2, 91.1)
- removed the R142 at (135.2, 133.1)
- removed the R142 at (78.2, 133.1)
- removed the R143 at (133.0, 130.5)
- removed the R143 at (76.0, 130.5)
- removed the R143 at (133.0, 88.5)
- removed the R143 at (76.0, 88.5)
- removed the R144 at (85.7, 85.4)
- removed the R144 at (85.7, 127.4)
- removed the R144 at (142.7, 85.4)
- removed the R144 at (142.7, 127.4)
- removed the R145 at (94.9, 123.8)
- removed the R145 at (94.9, 81.8)
- removed the R145 at (151.9, 81.8)
- removed the R145 at (151.9, 123.8)
- removed the R146 at (94.9, 124.8)
- removed the R146 at (151.9, 124.8)
- removed the R146 at (151.9, 82.8)
- removed the R146 at (94.9, 82.8)
- removed the R147 at (132.3, 66.4)
- removed the R147 at (132.3, 108.4)
- removed the R147 at (75.3, 66.4)
- removed the R147 at (75.3, 108.4)
- removed the R148 at (76.3, 108.4)
- removed the R148 at (76.3, 66.4)
- removed the R148 at (133.3, 66.4)
- removed the R148 at (133.3, 108.4)
- removed the R149 at (77.3, 108.4)
- removed the R149 at (134.3, 108.4)
- removed the R149 at (77.3, 66.4)
- removed the R149 at (134.3, 66.4)
- removed the R15 at (113.3, 105.7)
- removed the R15 at (56.3, 63.7)
- removed the R15 at (113.3, 63.7)
- removed the R15 at (56.3, 105.7)
- removed the R150 at (135.3, 66.4)
- removed the R150 at (78.3, 66.4)
- removed the R150 at (135.3, 108.4)
- removed the R150 at (78.3, 108.4)
- removed the R16 at (113.3, 65.8)
- removed the R16 at (56.3, 65.8)
- removed the R16 at (113.3, 107.8)
- removed the R16 at (56.3, 107.8)
- removed the R17 at (150.9, 86.0)
- removed the R17 at (93.9, 128.1)
- removed the R17 at (93.9, 86.0)
- removed the R17 at (150.9, 128.1)
- removed the R18 at (92.5, 85.6)
- removed the R18 at (92.5, 127.6)
- removed the R18 at (149.4, 85.6)
- removed the R18 at (149.4, 127.6)
- removed the R2 at (50.1, 64.9)
- removed the R2 at (107.1, 106.9)
- removed the R2 at (107.1, 64.9)
- removed the R2 at (50.1, 106.9)
- removed the R21 at (152.7, 84.9)
- removed the R21 at (95.7, 126.9)
- removed the R21 at (95.7, 84.9)
- removed the R21 at (152.7, 126.9)
- removed the R23 at (80.7, 83.9)
- removed the R23 at (80.7, 125.9)
- removed the R23 at (137.7, 83.9)
- removed the R23 at (137.7, 125.9)
- removed the R24 at (55.1, 137.1)
- removed the R24 at (55.1, 95.1)
- removed the R24 at (112.1, 137.1)
- removed the R24 at (112.1, 95.1)
- removed the R25 at (111.1, 95.1)
- removed the R25 at (111.1, 137.1)
- removed the R25 at (54.1, 95.1)
- removed the R25 at (54.1, 137.1)
- removed the R27 at (112.1, 135.1)
- removed the R27 at (112.1, 93.1)
- removed the R27 at (55.1, 135.1)
- removed the R27 at (55.1, 93.1)
- removed the R29 at (107.5, 96.7)
- removed the R29 at (50.5, 96.7)
- removed the R29 at (50.5, 138.7)
- removed the R29 at (107.5, 138.7)
- removed the R3 at (83.7, 103.4)
- removed the R3 at (83.7, 61.4)
- removed the R3 at (140.7, 61.4)
- removed the R3 at (140.7, 103.4)
- removed the R30 at (117.4, 129.5)
- removed the R30 at (117.4, 87.5)
- removed the R30 at (60.4, 87.5)
- removed the R30 at (60.4, 129.5)
- removed the R31 at (110.1, 95.1)
- removed the R31 at (110.1, 137.1)
- removed the R31 at (53.1, 137.1)
- removed the R31 at (53.1, 95.1)
- removed the R32 at (114.1, 95.1)
- removed the R32 at (114.1, 137.1)
- removed the R32 at (57.1, 95.1)
- removed the R32 at (57.1, 137.1)
- removed the R33 at (112.5, 83.6)
- removed the R33 at (55.5, 83.6)
- removed the R33 at (112.5, 125.6)
- removed the R33 at (55.5, 125.6)
- removed the R34 at (109.7, 130.9)
- removed the R34 at (52.7, 88.9)
- removed the R34 at (109.7, 88.9)
- removed the R34 at (52.7, 130.9)
- removed the R35 at (53.4, 135.1)
- removed the R35 at (53.4, 93.1)
- removed the R35 at (110.4, 93.1)
- removed the R35 at (110.4, 135.1)
- removed the R36 at (110.1, 91.9)
- removed the R36 at (53.1, 133.9)
- removed the R36 at (53.1, 91.9)
- removed the R36 at (110.1, 133.9)
- removed the R37 at (52.9, 83.6)
- removed the R37 at (52.9, 125.6)
- removed the R37 at (109.8, 83.6)
- removed the R37 at (109.8, 125.6)
- removed the R38 at (114.3, 91.1)
- removed the R38 at (57.3, 133.1)
- removed the R38 at (57.3, 91.1)
- removed the R38 at (114.3, 133.1)
- removed the R39 at (113.5, 129.8)
- removed the R39 at (56.5, 87.8)
- removed the R39 at (113.5, 87.8)
- removed the R39 at (56.5, 129.8)
- removed the R4 at (85.2, 103.6)
- removed the R4 at (142.2, 103.6)
- removed the R4 at (142.2, 61.6)
- removed the R4 at (85.2, 61.6)
- removed the R40 at (58.5, 87.8)
- removed the R40 at (115.5, 129.8)
- removed the R40 at (58.5, 129.8)
- removed the R40 at (115.5, 87.8)
- removed the R41 at (109.7, 132.9)
- removed the R41 at (52.7, 132.9)
- removed the R41 at (109.7, 90.9)
- removed the R41 at (52.7, 90.9)
- removed the R42 at (119.0, 130.1)
- removed the R42 at (119.0, 88.1)
- removed the R42 at (62.0, 130.1)
- removed the R42 at (62.0, 88.1)
- removed the R43 at (109.7, 131.9)
- removed the R43 at (52.7, 89.9)
- removed the R43 at (109.7, 89.9)
- removed the R43 at (52.7, 131.9)
- removed the R44 at (135.1, 134.0)
- removed the R44 at (78.1, 134.0)
- removed the R44 at (135.1, 92.0)
- removed the R44 at (78.1, 92.0)
- removed the R45 at (79.1, 134.0)
- removed the R45 at (79.1, 92.0)
- removed the R45 at (136.1, 134.0)
- removed the R45 at (136.1, 92.0)
- removed the R46 at (79.0, 138.7)
- removed the R46 at (79.0, 96.7)
- removed the R46 at (136.0, 138.7)
- removed the R46 at (136.0, 96.7)
- removed the R47 at (77.7, 138.5)
- removed the R47 at (134.7, 96.5)
- removed the R47 at (77.7, 96.5)
- removed the R47 at (134.7, 138.5)
- removed the R48 at (76.7, 130.7)
- removed the R48 at (133.7, 88.7)
- removed the R48 at (76.7, 88.7)
- removed the R48 at (133.7, 130.7)
- removed the R5 at (50.2, 69.4)
- removed the R5 at (50.2, 111.4)
- removed the R5 at (107.2, 111.4)
- removed the R5 at (107.2, 69.4)
- removed the R50 at (128.9, 136.5)
- removed the R50 at (128.9, 94.5)
- removed the R50 at (71.9, 136.5)
- removed the R50 at (71.9, 94.5)
- removed the R51 at (74.3, 135.7)
- removed the R51 at (74.3, 93.7)
- removed the R51 at (131.3, 93.7)
- removed the R51 at (131.3, 135.7)
- removed the R54 at (72.1, 129.7)
- removed the R54 at (72.1, 87.7)
- removed the R54 at (129.1, 129.7)
- removed the R54 at (129.1, 87.7)
- removed the R55 at (132.7, 130.7)
- removed the R55 at (75.7, 88.7)
- removed the R55 at (75.7, 130.7)
- removed the R55 at (132.7, 88.7)
- removed the R58 at (78.7, 138.5)
- removed the R58 at (135.7, 96.5)
- removed the R58 at (78.7, 96.5)
- removed the R58 at (135.7, 138.5)
- removed the R59 at (84.2, 85.2)
- removed the R59 at (141.2, 127.2)
- removed the R59 at (141.2, 85.2)
- removed the R59 at (84.2, 127.2)
- removed the R6 at (49.2, 111.4)
- removed the R6 at (49.2, 69.4)
- removed the R6 at (106.2, 111.4)
- removed the R6 at (106.2, 69.4)
- removed the R61 at (79.0, 94.8)
- removed the R61 at (136.0, 136.8)
- removed the R61 at (79.0, 136.8)
- removed the R61 at (136.0, 94.8)
- removed the R62 at (87.5, 131.6)
- removed the R62 at (144.4, 131.6)
- removed the R62 at (144.4, 89.6)
- removed the R62 at (87.5, 89.6)
- removed the R63 at (85.8, 127.2)
- removed the R63 at (142.8, 85.2)
- removed the R63 at (142.8, 127.2)
- removed the R63 at (85.8, 85.2)
- removed the R64 at (144.4, 127.2)
- removed the R64 at (87.4, 127.2)
- removed the R64 at (87.4, 85.2)
- removed the R64 at (144.4, 85.2)
- removed the R65 at (146.0, 85.2)
- removed the R65 at (146.0, 127.2)
- removed the R65 at (89.0, 127.2)
- removed the R65 at (89.0, 85.2)
- removed the R66 at (152.1, 74.5)
- removed the R66 at (95.1, 116.5)
- removed the R66 at (95.1, 74.5)
- removed the R66 at (152.1, 116.5)
- removed the R67 at (94.8, 75.8)
- removed the R67 at (151.8, 117.8)
- removed the R67 at (151.8, 75.8)
- removed the R67 at (94.8, 117.8)
- removed the R7 at (134.4, 131.6)
- removed the R7 at (77.4, 131.6)
- removed the R7 at (77.4, 89.6)
- removed the R7 at (134.4, 89.6)
- removed the R70 at (147.4, 120.7)
- removed the R70 at (147.4, 78.7)
- removed the R70 at (90.4, 78.7)
- removed the R70 at (90.4, 120.7)
- removed the R71 at (89.4, 120.7)
- removed the R71 at (146.4, 120.7)
- removed the R71 at (146.4, 78.7)
- removed the R71 at (89.4, 78.7)
- removed the R72 at (88.4, 78.7)
- removed the R72 at (145.4, 120.7)
- removed the R72 at (88.4, 120.7)
- removed the R72 at (145.4, 78.7)
- removed the R73 at (87.4, 120.7)
- removed the R73 at (87.4, 78.7)
- removed the R73 at (144.4, 78.7)
- removed the R73 at (144.4, 120.7)
- removed the R78 at (92.6, 78.7)
- removed the R78 at (149.6, 120.7)
- removed the R78 at (92.6, 120.7)
- removed the R78 at (149.6, 78.7)
- removed the R79 at (91.4, 120.7)
- removed the R79 at (91.4, 78.7)
- removed the R79 at (148.4, 78.7)
- removed the R79 at (148.4, 120.7)
- removed the R8 at (135.4, 130.3)
- removed the R8 at (78.4, 130.3)
- removed the R8 at (78.4, 88.3)
- removed the R8 at (135.4, 88.3)
- removed the R84 at (84.0, 70.3)
- removed the R84 at (141.1, 112.3)
- removed the R84 at (141.1, 70.3)
- removed the R84 at (84.0, 112.3)
- removed the R85 at (141.1, 113.3)
- removed the R85 at (84.0, 113.3)
- removed the R85 at (84.0, 71.3)
- removed the R85 at (141.1, 71.3)
- removed the R86 at (90.5, 85.2)
- removed the R86 at (147.6, 127.2)
- removed the R86 at (147.6, 85.2)
- removed the R86 at (90.5, 127.2)
- removed the R87 at (92.1, 127.2)
- removed the R87 at (149.1, 127.2)
- removed the R87 at (92.1, 85.2)
- removed the R87 at (149.1, 85.2)
- removed the R88 at (150.7, 127.2)
- removed the R88 at (93.7, 127.2)
- removed the R88 at (93.7, 85.2)
- removed the R88 at (150.7, 85.2)
- removed the R89 at (83.9, 114.3)
- removed the R89 at (140.9, 72.3)
- removed the R89 at (83.9, 72.3)
- removed the R89 at (140.9, 114.3)
- removed the R9 at (84.1, 122.9)
- removed the R9 at (141.1, 122.9)
- removed the R9 at (141.1, 80.9)
- removed the R9 at (84.1, 80.9)
- removed the R90 at (140.9, 73.3)
- removed the R90 at (83.9, 73.3)
- removed the R90 at (140.9, 115.3)
- removed the R90 at (83.9, 115.3)
- removed the R91 at (83.9, 74.3)
- removed the R91 at (140.9, 116.3)
- removed the R91 at (140.9, 74.3)
- removed the R91 at (83.9, 116.3)
- removed the R92 at (83.9, 75.3)
- removed the R92 at (140.9, 75.3)
- removed the R92 at (83.9, 117.3)
- removed the R92 at (140.9, 117.3)
- removed the R93 at (83.9, 119.3)
- removed the R93 at (140.9, 77.3)
- removed the R93 at (140.9, 119.3)
- removed the R93 at (83.9, 77.3)
- removed the R94 at (83.9, 118.3)
- removed the R94 at (140.9, 76.3)
- removed the R94 at (83.9, 76.3)
- removed the R94 at (140.9, 118.3)
- removed the R95 at (95.3, 85.2)
- removed the R95 at (152.3, 127.2)
- removed the R95 at (152.3, 85.2)
- removed the R95 at (95.3, 127.2)
- removed the R96 at (94.8, 76.8)
- removed the R96 at (151.8, 76.8)
- removed the R96 at (151.8, 118.8)
- removed the R96 at (94.8, 118.8)
- removed the R97 at (91.0, 78.7)
- removed the R97 at (148.0, 120.7)
- removed the R97 at (148.0, 78.7)
- removed the R97 at (91.0, 120.7)
- removed the R98 at (147.0, 78.7)
- removed the R98 at (147.0, 120.7)
- removed the R98 at (90.0, 120.7)
- removed the R98 at (90.0, 78.7)
- removed the R99 at (89.0, 78.7)
- removed the R99 at (146.0, 78.7)
- removed the R99 at (146.0, 120.7)
- removed the R99 at (89.0, 120.7)
- removed the SW1 at (104.3, 88.7)
- removed the SW1 at (104.3, 130.7)
- removed the SW1 at (47.3, 130.7)
- removed the SW1 at (47.3, 88.7)
- removed the TP1 at (140.2, 101.3)
- removed the TP1 at (83.2, 59.4)
- removed the TP1 at (83.2, 101.3)
- removed the TP1 at (140.2, 59.4)
- removed the TP10 at (86.9, 83.5)
- removed the TP10 at (86.9, 125.5)
- removed the TP10 at (143.9, 83.5)
- removed the TP10 at (143.9, 125.5)
- removed the TP11 at (90.8, 132.6)
- removed the TP11 at (147.8, 90.6)
- removed the TP11 at (90.8, 90.6)
- removed the TP11 at (147.8, 132.6)
- removed the TP12 at (62.1, 83.7)
- removed the TP12 at (119.1, 125.7)
- removed the TP12 at (62.1, 125.7)
- removed the TP12 at (119.1, 83.7)
- removed the TP2 at (50.6, 71.8)
- removed the TP2 at (107.6, 71.8)
- removed the TP2 at (50.6, 113.8)
- removed the TP2 at (107.6, 113.8)
- removed the TP3 at (54.4, 105.3)
- removed the TP3 at (111.4, 105.3)
- removed the TP3 at (54.4, 63.3)
- removed the TP3 at (111.4, 63.3)
- removed the TP4 at (151.9, 87.6)
- removed the TP4 at (94.9, 129.6)
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Other:
- board text added: "Created on 2026-08-20"
- board text removed: "Created on 2026-07-12"
